Commit message: Update NexArm simulation assets and documentation
Add complete workflow steps to README
Fix gripper joint directions and positions in MuJoCo models
Update collision geometry and physics parameters
Add gripper class defaults and improve table positioning
Add jaw position tracking in pick-place task
Add gripper geometry assertions to tests

File: sim/mobile_nexarm/generated/mobile_bi_nexarm.urdf (robot description, URDF)
Before this commit: robot mobile_bi_nexarm, 21 links, 20 joints
Links:
- added link left_gripper_base
- added link right_gripper_base
Joints:
- added joint left_gripper_base_joint: type fixed, parent left_link_5, child left_gripper_base, origin xyz=0 0.06 0 rpy=0 0 0
- added joint right_gripper_base_joint: type fixed, parent right_link_5, child right_gripper_base, origin xyz=0 0.06 0 rpy=0 0 0
- joint left_elbow_flex: origin xyz=0 0.08 0 rpy=0 0 0 -> xyz=0 0.19 0 rpy=0 0 0
- joint left_gripper: axis 1 0 0 -> -1 0 0; limit lower=-0.0255 upper=0.0 effort=100 velocity=3 -> lower=-0.0255 upper=0.0 effort=100 velocity=0.1; origin xyz=0 0.08 0 rpy=0 0 0 -> xyz=0.017 0 0 rpy=0 0 0; parent left_link_5 -> left_gripper_base
- joint left_gripper_mimic: axis 1 0 0 -> -1 0 0; origin (none) -> xyz=-0.017 0 0 rpy=0 0 0; parent left_gripper -> left_gripper_base
- joint left_shoulder_pan: origin xyz=0 0.08 0 rpy=0 0 0 -> xyz=0 0 0 rpy=0 0 0
- joint left_wrist_flex: origin xyz=0 0.08 0 rpy=0 0 0 -> xyz=0 0.15 0 rpy=0 0 0
- joint left_wrist_roll: origin xyz=0 0.08 0 rpy=0 0 0 -> xyz=0 0.07 0 rpy=0 0 0
- joint right_elbow_flex: origin xyz=0 0.08 0 rpy=0 0 0 -> xyz=0 0.19 0 rpy=0 0 0
- joint right_gripper: axis 1 0 0 -> -1 0 0; limit lower=-0.0255 upper=0.0 effort=100 velocity=3 -> lower=-0.0255 upper=0.0 effort=100 velocity=0.1; origin xyz=0 0.08 0 rpy=0 0 0 -> xyz=0.017 0 0 rpy=0 0 0; parent right_link_5 -> right_gripper_base
- joint right_gripper_mimic: axis 1 0 0 -> -1 0 0; origin (none) -> xyz=-0.017 0 0 rpy=0 0 0; parent right_gripper -> right_gripper_base
- joint right_shoulder_pan: origin xyz=0 0.08 0 rpy=0 0 0 -> xyz=0 0 0 rpy=0 0 0
- joint right_wrist_flex: origin xyz=0 0.08 0 rpy=0 0 0 -> xyz=0 0.15 0 rpy=0 0 0
- joint right_wrist_roll: origin xyz=0 0.08 0 rpy=0 0 0 -> xyz=0 0.07 0 rpy=0 0 0
